Commit message: use interpolated trajs as expert_demos; refactor such that expert demos only contain keypoints/no joint state

File: mbirl/env/kuka_iiwa/urdf/iiwa7_ft_with_obj_keypts.urdf (robot description, URDF)
Before this commit: robot iiwa7, 12 links, 11 joints
Links:
- added link iiwa_link_ee, mass 0
Joints:
- joint iiwa_joint_ee: parent iiwa_link_fts -> iiwa_link_ee

Commit message: irl working with RBF weights

File: mbirl/env/kuka_iiwa/urdf/iiwa7_ft_with_obj_keypts.urdf (robot description, URDF)
Before this commit: robot iiwa7, 13 links, 11 joints
Links:
- removed link iiwa_link_ee
Joints:
- removed joint iiwa_joint_ee
- added joint keypoint_3: type fixed, parent kp_link_2, child kp_link_3, origin xyz=0 0.0 0.05 rpy=0 0 0
- joint keypoint_1: child kp_link_2 -> kp_link_1; origin xyz=0 0.0 0.05 rpy=0 0 0 -> xyz=0 0 0.05 rpy=0 0 0; parent kp_link_3 -> iiwa_link_fts
- joint keypoint_2: child kp_link_1 -> kp_link_2; parent kp_link_2 -> kp_link_1
